File: kicad/spectrum.kicad_sch (KiCad schematic)
At the start: 247 parts, among them J1 Micro USB B, J2 Input, J3 Output, SW1 POWER, SW2 RIGHT SOURCE, SW3 LEFT SOURCE, U1 LM833, U10 LM833, U11 LM833, U12 LM833, U13 LM833, U14 LM833, U15 LM833, U16 LM833, U17 LM833, U18 LM833, U19 LM833, U2 LM833, U20 LM833, U21 LM833, U22 LM833, U23 L7805, U3 LM833, U4 LM833, U5 LM833, U6 LM833, U7 LM833, U8 LM833, U9 LM833

Commit message: Test points
Parts:
- removed SW1: POWER, symbol Switch:SW_SPST
- added SW1: RIGHT SOURCE, symbol Switch:SW_SPDT
- added TP1: +5V, symbol Connector:TestPoint
- added TP10, TP24: 125Hz, symbol Connector:TestPoint
- added TP11, TP25: 63Hz, symbol Connector:TestPoint
- added TP12, TP26: 31.5Hz, symbol Connector:TestPoint
- added TP13: Vout_L, symbol Connector:TestPoint
- added TP14: GND, symbol Connector:TestPoint
- added TP15: VGND, symbol Connector:TestPoint
- added TP16: Vout_R, symbol Connector:TestPoint
- added TP17, TP3: 16kHz, symbol Connector:TestPoint
- added TP18, TP4: 8kHz, symbol Connector:TestPoint
- added TP19, TP5: 4kHz, symbol Connector:TestPoint
- added TP2: Vin_L, symbol Connector:TestPoint
- added TP20, TP6: 2kHz, symbol Connector:TestPoint
- added TP21, TP7: 1kHz, symbol Connector:TestPoint
- added TP22, TP8: 500Hz, symbol Connector:TestPoint
- added TP23, TP9: 250Hz, symbol Connector:TestPoint
- added TP27: Vin_R, symbol Connector:TestPoint
Connections:
- net +5V: now also TP1.1
- net GNDREF: now also TP14.1
- net VGND: now also TP15.1
- net Vin_L: now also TP2.1; no longer C50.1
- net Vin_R: now also C50.1, TP27.1
- net Vout_L: now also TP13.1; no longer C29.2
- net Vout_R: now also C29.2, TP16.1
- net at PTL6.2, PTL6.3, R46.2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: now also TP7.1
- net at PTL40.2, PTL40.3, R84.2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: now also TP25.1
- net at PTL32.2, PTL32.3, R76.2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: now also TP17.1
- net at PTL10.2, PTL10.3, R50.2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: now also TP11.1
- net at PTL11.2, PTL11.3, R51.2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: now also TP12.1
- net at PTL9.2, PTL9.3, R49.2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: now also TP10.1
- net at PTL41.2, PTL41.3, R85.2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: now also TP26.1
- net at PTL3.2, PTL3.3, R43.2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: now also TP4.1
- net at PTL7.2, PTL7.3, R47.2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: now also TP8.1
- net at PTL8.2, PTL8.3, R48.2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: now also TP9.1
- net at PTL5.2, PTL5.3, R45.2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: now also TP6.1
- net at PTL37.2, PTL37.3, R81.2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: now also TP22.1
- net at J1.1 (VBUS): now also SW1.2 (B)
- net at PTL2.2, PTL2.3, R42.2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: now also TP3.1
- net at PTL34.2, PTL34.3, R78.2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: now also TP19.1
- net at PTL4.2, PTL4.3, R44.2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: now also TP5.1
- net at PTL35.2, PTL35.3, R79.2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: now also TP20.1
- net at PTL38.2, PTL38.3, R82.2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: now also TP23.1
- net at PTL39.2, PTL39.3, R83.2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: now also TP24.1
- net at PTL33.2, PTL33.3, R77.2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: now also TP18.1
- net at PTL36.2, PTL36.3, R80.2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: now also TP21.1
- net at U23.1 (IN): now also SW1.1 (A)
Other:
- moved on the sheet: C23, C24, C25, C26, C27, C28, J1, J2, J3, R63, R64, SW2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

Commit message: Switch to USB-A
Parts:
- removed J1: Micro USB B, symbol Connector:USB_B_Micro
- added J1: USB_A, symbol Connector:USB_A
- PTL1, PTL42: value 100K -> 10K
- R1, R126: value 1K -> 100R
- SW1: value RIGHT SOURCE -> POWER
Connections:
- net GNDREF: now also J1.4 (GND), J1.5 (Shield)
- net at SW1.2 (B): now also J1.1 (VBUS)
Changed lines of the file:
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@@
     (in_bom yes) (on_board yes)
     (property "Reference" "PTL42" (id 0) (at 534.67 194.31 90))
-    (property "Value" "100K" (id 1) (at 530.86 199.39 90))
+    (property "Value" "10K" (id 1) (at 530.86 199.39 90))
     (property "Footprint" "" (id 2) (at 530.86 196.85 0)
       (effects (font (size 1.27 1.27)) hide)
@@
     (pin "5")
   )
-  (symbol (lib_id "Connector:USB_B_Micro") (at 256.54 97.79 0) (unit 1)
-    (in_bom yes) (on_board yes) (fields_autoplaced)
-    (property "Reference" "J1" (id 0) (at 256.54 85.09 0))
-    (property "Value" "Micro USB B" (id 1) (at 256.54 87.63 0))
-    (property "Footprint" "" (id 2) (at 260.35 99.06 0)
-      (effects (font (size 1.27 1.27)) hide)
-    )
-    (property "Datasheet" "~" (id 3) (at 260.35 99.06 0)
-      (effects (font (size 1.27 1.27)) hide)
-    )
-    (pin "1")
-    (pin "2")
-    (pin "3")
-    (pin "4")
-    (pin "5")
-    (pin "6")
-  )
   (symbol (lib_id "bourns_ptl:Bourns_PTL") (at 443.23 302.26 270) (mirror x) (unit 2)
     (in_bom yes) (on_board yes)
@@
     (in_bom yes) (on_board yes)
     (property "Reference" "R126" (id 0) (at 547.37 201.93 90))
-    (property "Value" "1K" (id 1) (at 547.37 207.01 90))
+    (property "Value" "100R" (id 1) (at 547.37 207.01 90))
     (property "Footprint" "" (id 2) (at 547.624 205.486 90)
       (effects (font (size 1.27 1.27)) hide)
@@
     (in_bom yes) (on_board yes)
     (property "Reference" "SW1" (id 0) (at 271.78 88.9 0))
-    (property "Value" "RIGHT SOURCE" (id 1) (at 274.32 97.79 0))
+    (property "Value" "POWER" (id 1) (at 271.78 97.79 0))
     (property "Footprint" "" (id 2) (at 271.78 92.71 0)
       (effects (font (size 1.27 1.27)) hide)
@@
     (pin "3")
   )
+  (symbol (lib_id "Connector:USB_A") (at 256.54 97.79 0) (unit 1)
+    (in_bom yes) (on_board yes) (fields_autoplaced)
+    (property "Reference" "J1" (id 0) (at 256.54 85.09 0))
+    (property "Value" "USB_A" (id 1) (at 256.54 87.63 0))
+    (property "Footprint" "" (id 2) (at 260.35 99.06 0)
+      (effects (font (size 1.27 1.27)) hide)
+    )
+    (property "Datasheet" " ~" (id 3) (at 260.35 99.06 0)
+      (effects (font (size 1.27 1.27)) hide)
+    )
+    (pin "1")
+    (pin "2")
+    (pin "3")
+    (pin "4")
+    (pin "5")
+  )
   (symbol (lib_id "Device:R_US") (at 99.06 199.39 0) (unit 1)
     (in_bom yes) (on_board yes)
@@
     (in_bom yes) (on_board yes)
     (property "Reference" "PTL1" (id 0) (at 63.5 194.31 90))
-    (property "Value" "100K" (id 1) (at 67.31 199.39 90))
+    (property "Value" "10K" (id 1) (at 67.31 199.39 90))
     (property "Footprint" "" (id 2) (at 67.31 196.85 0)
       (effects (font (size 1.27 1.27)) hide)
@@
     (in_bom yes) (on_board yes)
     (property "Reference" "R1" (id 0) (at 50.8 201.93 90))
-    (property "Value" "1K" (id 1) (at 50.8 207.01 90))
+    (property "Value" "100R" (id 1) (at 50.8 207.01 90))
     (property "Footprint" "" (id 2) (at 50.546 205.486 90)
       (effects (font (size 1.27 1.27)) hide)
@@
       (reference "C50") (unit 1) (value "470uF") (footprint "")
     )
-    (path "/40cbc0de-ba23-461b-bccc-b38c5108c933"
-      (reference "J1") (unit 1) (value "Micro USB B") (footprint "")
+    (path "/bd171de3-4d48-49a8-a351-111a8a1d6d82"
+      (reference "J1") (unit 1) (value "USB_A") (footprint "")
     )
     (path "/0831003e-d566-49ce-9e20-3d4987641f44"
@@
     )
     (path "/c7441e37-7730-484c-998d-621798e77c2a"
-      (reference "PTL1") (unit 2) (value "100K") (footprint "")
+      (reference "PTL1") (unit 2) (value "10K") (footprint "")
     )
     (path "/48ea81c8-42db-48c8-bbe4-8eaf13d3b35f"
@@
     )
     (path "/22156359-44e1-4a95-bb07-6494a2c04c71"
-      (reference "PTL42") (unit 2) (value "100K") (footprint "")
+      (reference "PTL42") (unit 2) (value "10K") (footprint "")
     )
     (path "/e080946b-11f2-49f7-a907-a5898cf531fe"
-      (reference "R1") (unit 1) (value "1K") (footprint "")
+      (reference "R1") (unit 1) (value "100R") (footprint "")
     )
     (path "/cb2e50f6-8c65-43f2-b38d-30223dcabf92"
@@
     )
     (path "/85634b21-e966-40ed-a4d2-e59f53fee5db"
-      (reference "R126") (unit 1) (value "1K") (footprint "")
+      (reference "R126") (unit 1) (value "100R") (footprint "")
     )
     (path "/b58d0db8-9a2f-40d6-80cd-7939e1b77f51"
-      (reference "SW1") (unit 1) (value "RIGHT SOURCE") (footprint "")
+      (reference "SW1") (unit 1) (value "POWER") (footprint "")
     )
     (path "/54b58231-31cf-475e-a2c6-f37f98e7bb7c"

Commit message: Increase preamp input resistor to 1K
Parts:
- R1, R126: value 100R -> 1K
Changed lines of the file:
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@@
     (in_bom yes) (on_board yes)
     (property "Reference" "R126" (id 0) (at 547.37 201.93 90))
-    (property "Value" "100R" (id 1) (at 547.37 207.01 90))
+    (property "Value" "1K" (id 1) (at 547.37 207.01 90))
     (property "Footprint" "" (id 2) (at 547.624 205.486 90)
       (effects (font (size 1.27 1.27)) hide)
@@
     (in_bom yes) (on_board yes)
     (property "Reference" "R1" (id 0) (at 50.8 201.93 90))
-    (property "Value" "100R" (id 1) (at 50.8 207.01 90))
+    (property "Value" "1K" (id 1) (at 50.8 207.01 90))
     (property "Footprint" "" (id 2) (at 50.546 205.486 90)
       (effects (font (size 1.27 1.27)) hide)
@@
     )
     (path "/e080946b-11f2-49f7-a907-a5898cf531fe"
-      (reference "R1") (unit 1) (value "100R") (footprint "")
+      (reference "R1") (unit 1) (value "1K") (footprint "")
     )
     (path "/cb2e50f6-8c65-43f2-b38d-30223dcabf92"
@@
     )
     (path "/85634b21-e966-40ed-a4d2-e59f53fee5db"
-      (reference "R126") (unit 1) (value "100R") (footprint "")
+      (reference "R126") (unit 1) (value "1K") (footprint "")
     )
     (path "/b58d0db8-9a2f-40d6-80cd-7939e1b77f51"

Commit message: Fix POT LEDs and use barrel jack for power
Parts:
- removed J1: USB_A, symbol Connector:USB_A
- removed PTL23, PTL24, PTL25, PTL26, PTL27, PTL28, PTL29, PTL30, PTL31: LED, symbol bourns_ptl:Bourns_PTL
- added J1: SUPPLY, symbol Connector:Barrel_Jack
- added unit 1 of PTL1
- added unit 1 of PTL12
- added unit 1 of PTL13
- added unit 1 of PTL14
- added unit 1 of PTL15
- added unit 1 of PTL16
- added unit 1 of PTL17
- added unit 1 of PTL18
- added unit 1 of PTL19
- added unit 1 of PTL20
- added unit 1 of PTL21
- added R127: 1K, symbol Device:R_US
- added R128: 5.6K, symbol Device:R_US
- PTL10: renamed from PTL19; value LED -> 10K
- PTL11: renamed from PTL21; value LED -> 10K
- PTL2: renamed from PTL12; value LED -> 10K
- PTL22: value LED -> 10K
- PTL3: renamed from PTL14; value LED -> 10K
- PTL4: renamed from PTL16; value LED -> 10K
- PTL5: renamed from PTL18; value LED -> 10K
- PTL6: renamed from PTL20; value LED -> 10K
- PTL7: renamed from PTL13; value LED -> 10K
- PTL8: renamed from PTL15; value LED -> 10K
- PTL9: renamed from PTL17; value LED -> 10K
- R65: value 1K -> 5.6K
- renumbered PTL42 to PTL12, PTL32 to PTL13, PTL33 to PTL14, PTL34 to PTL15, PTL35 to PTL16, PTL36 to PTL17, PTL37 to PTL18, PTL38 to PTL19, PTL39 to PTL20, PTL40 to PTL21, PTL41 to PTL22, U9 to U10, U15 to U14, U17 to U15, U19 to U16, U21 to U17, U14 to U18, U16 to U19, U18 to U20, U20 to U21, U4 to U3, U6 to U4, U8 to U5, U10 to U6, U3 to U7, U5 to U8, U7 to U9
Connections:
- net +5V: now also R127.1, R128.1
- net GNDREF: now also J1.2, PTL1.5 (E), PTL12.5 (E), PTL13.5 (E), PTL14.5 (E), PTL15.5 (E), PTL16.5 (E), PTL17.5 (E), PTL18.5 (E), PTL19.5 (E), PTL20.5 (E), PTL21.5 (E)
- net at R70.2: now also PTL15.4 (B)
- net at R67.2: now also PTL18.4 (B)
- net at PTL22.4 (B): now also R127.2; no longer R65.2
- net at R74.2: now also PTL21.4 (B)
- net at R69.2: now also PTL19.4 (B)
- net at R66.2: now also PTL13.4 (B)
- net at R71.2: now also PTL20.4 (B)
- net at R72.2: now also PTL16.4 (B)
- net at R75.2: now also PTL17.4 (B)
- net at SW1.2 (B): now also SW1.3 (C), J1.1
- net at R68.2: now also PTL14.4 (B)
- new net: PTL1.4 (B), R65.2
- new net: PTL12.4 (B), R128.2
Other:
- moved on the sheet: C23, C24, C25, C26, C27, C28, PTL10A, PTL11A, PTL2A, PTL3A, PTL4A, PTL5A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

Commit message: Footprints
Parts:
- C1, C22, C23, C25, C26, C29, C50: footprint (none) -> Capacitor_THT:CP_Radial_D8.0mm_P3.50mm
- C10, C11, C12, C13, C14, C15, C16, C17, C18, C19, C2, C20, C21, C24, C27, C28, C3, C30, C31, C32, C33, C34, C35, C36, C37, C38, C39, C4, C40, C41, C42, C43, C44, C45, C46, C47, C48, C49, C5, C6, C7, C8, C9: footprint (none) -> Capacitor_THT:C_Disc_D4.3mm_W1.9mm_P5.00mm
- J1: footprint (none) -> Connector_BarrelJack:BarrelJack_Horizontal
- J2, J3: footprint (none) -> Audio_Jack_STX35013N:STX35013N
- PTL1, PTL10, PTL11, PTL12, PTL13, PTL14, PTL15, PTL16, PTL17, PTL18, PTL19, PTL2, PTL20, PTL21, PTL22, PTL3, PTL4, PTL5, PTL6, PTL7, PTL8, PTL9: footprint (none) -> Bourns_PTL:PTL30
- R1, R10, R100, R101, R102, R103, R104, R105, R106, R107, R108, R109, R11, R110, R111, R112, R113, R114, R115, R116, R117, R118, R119, R12, R120, R121, R122, R123, R124, R125, R126, R127, R128, R13, R14, R15, R16, R17, R18, R19, R2, R20, R21, R22, R23, R24, R25, R26, R27, R28, R29, R3, R30, R31, R32, R33, R34, R35, R36, R37, R38, R39, R4, R40, R41, R42, R43, R44, R45, R46, R47, R48, R49, R5, R50, R51, R52, R53, R54, R55, R56, R57, R58, R59, R6, R60, R61, R62, R63, R64, R65, R66, R67, R68, R69, R7, R70, R71, R72, R73, R74, R75, R76, R77, R78, R79, R8, R80, R81, R82, R83, R84, R85, R86, R87, R88, R89, R9, R90, R91, R92, R93, R94, R95, R96, R97, R98, R99: footprint (none) -> Resistor_THT:R_Axial_DIN0207_L6.3mm_D2.5mm_P7.62mm_Horizontal
- SW1, SW2, SW3: footprint (none) -> CK_Switches:SW_1101M2S3CQE2
- TP1, TP10, TP11, TP12, TP13, TP14, TP15, TP16, TP17, TP18, TP19, TP2, TP20, TP21, TP22, TP23, TP24, TP25, TP26, TP27, TP3, TP4, TP5, TP6, TP7, TP8, TP9: footprint (none) -> TestPoint:TestPoint_Keystone_5000-5004_Miniature
- U1, U10, U11, U12, U13, U14, U15, U16, U17, U18, U19, U2, U20, U21, U22, U3, U4, U5, U6, U7, U8, U9: footprint (none) -> Package_DIP:DIP-8_W7.62mm_Socket_LongPads
- U23: footprint (none) -> Package_TO_SOT_THT:TO-220-3_Vertical

Commit message: Filter array component layout
Parts:
- added TP28: Vpreamp_L, TestPoint:TestPoint_Keystone_5000-5004_Miniature, symbol Connector:TestPoint
- added TP29: Vpreamp_R, TestPoint:TestPoint_Keystone_5000-5004_Miniature, symbol Connector:TestPoint
Connections:
- net Vin_L: now also C1.2, R1.2; no longer C1.1, J2.T
- net Vin_R: now also C50.2, R126.2; no longer C50.1, J2.R
- net at PTL12.2, PTL12.3, R116.2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: now also TP29.1
- net at PTL1.2, PTL1.3, R10.2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: now also TP28.1
- new net Vsrc_L: C1.1, J2.T
- new net Vsrc_R: C50.1, J2.R
Other:
- moved on the sheet: C1, C50, TP2, TP27

Commit message: Fix bypass routes
Connections:
- net Vsrc_L is gone; now on net Vin_L: C1.1, J2.T
- net Vsrc_R is gone; now on net Vin_R: C50.1, J2.R
- net Vin_L: no longer C1.2, R1.2
- net Vin_R: no longer C50.2, R126.2
- new net: C50.2, R126.2
- new net: C1.2, R1.2
Other:
- moved on the sheet: C1, C50, TP2, TP27

Commit message: More component layout
Connections:
- net VGND: now also U1.3 (+), U1.5 (+); no longer U1.3 (+), U1.5 (+)
- net at R42.1, R43.1, R44.1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: now also U1.2 (-); no longer U1.6 (-)
- net at C22.1, R54.1: now also U1.1; no longer U1.7
- net at PTL1.2, PTL1.3, R10.2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: now also U1.7; no longer U1.1
- net at PTL1.1, R1.1: now also U1.6 (-); no longer U1.2 (-)
Changed lines of the file:
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@@
     (pin "2")
   )
-  (symbol (lib_id "Device:Opamp_Dual") (at 201.93 209.55 0) (mirror x) (unit 2)
+  (symbol (lib_id "Device:Opamp_Dual") (at 201.93 209.55 0) (mirror x) (unit 1)
     (in_bom yes) (on_board yes)
     (property "Reference" "U1" (id 0) (at 201.93 214.63 0))
@@
       (effects (font (size 1.27 1.27)) hide)
     )
+    (pin "1")
+    (pin "2")
+    (pin "3")
+  )
+  (symbol (lib_id "Device:R_US") (at 347.98 165.1 0) (mirror y) (unit 1)
+    (in_bom yes) (on_board yes)
+    (property "Reference" "R67" (id 0) (at 344.17 163.83 0))
+    (property "Value" "1K" (id 1) (at 344.17 166.37 0))
+    (property "Footprint" "Resistor_THT:R_Axial_DIN0207_L6.3mm_D2.5mm_P7.62mm_Horizontal" (id 2) (at 346.964 165.354 90)
+      (effects (font (size 1.27 1.27)) hide)
+    )
+    (property "Datasheet" "~" (id 3) (at 347.98 165.1 0)
+      (effects (font (size 1.27 1.27)) hide)
+    )
+    (pin "1")
+    (pin "2")
+  )
+  (symbol (lib_id "Device:R_US") (at 99.06 140.97 0) (unit 1)
+    (in_bom yes) (on_board yes)
+    (property "Reference" "R14" (id 0) (at 100.33 139.7 0)
+      (effects (font (size 1.27 1.27)) (justify left))
+    )
+    (property "Value" "200R" (id 1) (at 100.33 142.24 0)
+      (effects (font (size 1.27 1.27)) (justify left))
+    )
+    (property "Footprint" "Resistor_THT:R_Axial_DIN0207_L6.3mm_D2.5mm_P7.62mm_Horizontal" (id 2) (at 100.076 141.224 90)
+      (effects (font (size 1.27 1.27)) hide)
+    )
+    (property "Datasheet" "~" (id 3) (at 99.06 140.97 0)
+      (effects (font (size 1.27 1.27)) hide)
+    )
+    (pin "1")
+    (pin "2")
+  )
+  (symbol (lib_id "Device:Opamp_Dual") (at 476.25 224.79 180) (unit 1)
+    (in_bom yes) (on_board yes)
+    (property "Reference" "U18" (id 0) (at 476.25 229.87 0))
+    (property "Value" "LM833" (id 1) (at 476.25 232.41 0))
+    (property "Footprint" "Package_DIP:DIP-8_W7.62mm_Socket_LongPads" (id 2) (at 476.25 224.79 0)
+      (effects (font (size 1.27 1.27)) hide)
+    )
+    (property "Datasheet" "~" (id 3) (at 476.25 224.79 0)
+      (effects (font (size 1.27 1.27)) hide)
+    )
+    (pin "1")
+    (pin "2")
+    (pin "3")
+  )
+  (symbol (lib_id "Device:C_Polarized_Small_US") (at 379.73 209.55 270) (mirror x) (unit 1)
+    (in_bom yes) (on_board yes)
+    (property "Reference" "C29" (id 0) (at 378.46 207.01 90)
+      (effects (font (size 1.27 1.27)) (justify left))
+    )
+    (property "Value" "470uF" (id 1) (at 377.19 212.09 90)
+      (effects (font (size 1.27 1.27)) (justify left))
+    )
+    (property "Footprint" "Capacitor_THT:CP_Radial_D8.0mm_P3.50mm" (id 2) (at 379.73 209.55 0)
+      (effects (font (size 1.27 1.27)) hide)
+    )
+    (property "Datasheet" "~" (id 3) (at 379.73 209.55 0)
+      (effects (font (size 1.27 1.27)) hide)
+    )
+    (pin "1")
+    (pin "2")
+  )
+  (symbol (lib_id "power:GNDREF") (at 99.06 205.74 0) (unit 1)
+    (in_bom yes) (on_board yes) (fields_autoplaced)
+    (property "Reference" "#PWR0131" (id 0) (at 99.06 212.09 0)
+      (effects (font (size 1.27 1.27)) hide)
+    )
+    (property "Value" "GNDREF" (id 1) (at 99.06 210.82 0)
+      (effects (font (size 1.27 1.27)) hide)
+    )
+    (property "Footprint" "" (id 2) (at 99.06 205.74 0)
+      (effects (font (size 1.27 1.27)) hide)
+    )
+    (property "Datasheet" "" (id 3) (at 99.06 205.74 0)
+      (effects (font (size 1.27 1.27)) hide)
+    )
+    (pin "1")
+  )
+  (symbol (lib_id "power:+5V") (at 393.7 160.02 0) (mirror y) (unit 1)
+    (in_bom yes) (on_board yes)
+    (property "Reference" "#PWR0175" (id 0) (at 393.7 163.83 0)
+      (effects (font (size 1.27 1.27)) hide)
+    )
+    (property "Value" "+5V" (id 1) (at 392.43 156.21 0)
+      (effects (font (size 1.27 1.27)) (justify right))
+    )
+    (property "Footprint" "" (id 2) (at 393.7 160.02 0)
+      (effects (font (size 1.27 1.27)) hide)
+    )
+    (property "Datasheet" "" (id 3) (at 393.7 160.02 0)
+      (effects (font (size 1.27 1.27)) hide)
+    )
+    (pin "1")
+  )
+  (symbol (lib_id "Device:Opamp_Dual") (at 67.31 207.01 0) (mirror x) (unit 2)
+    (in_bom yes) (on_board yes)
+    (property "Reference" "U1" (id 0) (at 67.31 212.09 0))
+    (property "Value" "LM833" (id 1) (at 67.31 214.63 0))
+    (property "Footprint" "Package_DIP:DIP-8_W7.62mm_Socket_LongPads" (id 2) (at 67.31 207.01 0)
+      (effects (font (size 1.27 1.27)) hide)
+    )
+    (property "Datasheet" "~" (id 3) (at 67.31 207.01 0)
+      (effects (font (size 1.27 1.27)) hide)
+    )
     (pin "5")
     (pin "6")
     (pin "7")
-  )
-  (symbol (lib_id "Device:R_US") (at 347.98 165.1 0) (mirror y) (unit 1)
-    (in_bom yes) (on_board yes)
-    (property "Reference" "R67" (id 0) (at 344.17 163.83 0))
-    (property "Value" "1K" (id 1) (at 344.17 166.37 0))
-    (property "Footprint" "Resistor_THT:R_Axial_DIN0207_L6.3mm_D2.5mm_P7.62mm_Horizontal" (id 2) (at 346.964 165.354 90)
-      (effects (font (size 1.27 1.27)) hide)
-    )
-    (property "Datasheet" "~" (id 3) (at 347.98 165.1 0)
-      (effects (font (size 1.27 1.27)) hide)
-    )
-    (pin "1")
-    (pin "2")
-  )
-  (symbol (lib_id "Device:R_US") (at 99.06 140.97 0) (unit 1)
-    (in_bom yes) (on_board yes)
-    (property "Reference" "R14" (id 0) (at 100.33 139.7 0)
-      (effects (font (size 1.27 1.27)) (justify left))
-    )
-    (property "Value" "200R" (id 1) (at 100.33 142.24 0)
-      (effects (font (size 1.27 1.27)) (justify left))
-    )
-    (property "Footprint" "Resistor_THT:R_Axial_DIN0207_L6.3mm_D2.5mm_P7.62mm_Horizontal" (id 2) (at 100.076 141.224 90)
-      (effects (font (size 1.27 1.27)) hide)
-    )
-    (property "Datasheet" "~" (id 3) (at 99.06 140.97 0)
-      (effects (font (size 1.27 1.27)) hide)
-    )
-    (pin "1")
-    (pin "2")
-  )
-  (symbol (lib_id "Device:Opamp_Dual") (at 476.25 224.79 180) (unit 1)
-    (in_bom yes) (on_board yes)
-    (property "Reference" "U18" (id 0) (at 476.25 229.87 0))
-    (property "Value" "LM833" (id 1) (at 476.25 232.41 0))
-    (property "Footprint" "Package_DIP:DIP-8_W7.62mm_Socket_LongPads" (id 2) (at 476.25 224.79 0)
-      (effects (font (size 1.27 1.27)) hide)
-    )
-    (property "Datasheet" "~" (id 3) (at 476.25 224.79 0)
-      (effects (font (size 1.27 1.27)) hide)
-    )
-    (pin "1")
-    (pin "2")
-    (pin "3")
-  )
-  (symbol (lib_id "Device:C_Polarized_Small_US") (at 379.73 209.55 270) (mirror x) (unit 1)
-    (in_bom yes) (on_board yes)
-    (property "Reference" "C29" (id 0) (at 378.46 207.01 90)
-      (effects (font (size 1.27 1.27)) (justify left))
-    )
-    (property "Value" "470uF" (id 1) (at 377.19 212.09 90)
-      (effects (font (size 1.27 1.27)) (justify left))
-    )
-    (property "Footprint" "Capacitor_THT:CP_Radial_D8.0mm_P3.50mm" (id 2) (at 379.73 209.55 0)
-      (effects (font (size 1.27 1.27)) hide)
-    )
-    (property "Datasheet" "~" (id 3) (at 379.73 209.55 0)
-      (effects (font (size 1.27 1.27)) hide)
-    )
-    (pin "1")
-    (pin "2")
-  )
-  (symbol (lib_id "power:GNDREF") (at 99.06 205.74 0) (unit 1)
-    (in_bom yes) (on_board yes) (fields_autoplaced)
-    (property "Reference" "#PWR0131" (id 0) (at 99.06 212.09 0)
-      (effects (font (size 1.27 1.27)) hide)
-    )
-    (property "Value" "GNDREF" (id 1) (at 99.06 210.82 0)
-      (effects (font (size 1.27 1.27)) hide)
-    )
-    (property "Footprint" "" (id 2) (at 99.06 205.74 0)
-      (effects (font (size 1.27 1.27)) hide)
-    )
-    (property "Datasheet" "" (id 3) (at 99.06 205.74 0)
-      (effects (font (size 1.27 1.27)) hide)
-    )
-    (pin "1")
-  )
-  (symbol (lib_id "power:+5V") (at 393.7 160.02 0) (mirror y) (unit 1)
-    (in_bom yes) (on_board yes)
-    (property "Reference" "#PWR0175" (id 0) (at 393.7 163.83 0)
-      (effects (font (size 1.27 1.27)) hide)
-    )
-    (property "Value" "+5V" (id 1) (at 392.43 156.21 0)
-      (effects (font (size 1.27 1.27)) (justify right))
-    )
-    (property "Footprint" "" (id 2) (at 393.7 160.02 0)
-      (effects (font (size 1.27 1.27)) hide)
-    )
-    (property "Datasheet" "" (id 3) (at 393.7 160.02 0)
-      (effects (font (size 1.27 1.27)) hide)
-    )
-    (pin "1")
-  )
-  (symbol (lib_id "Device:Opamp_Dual") (at 67.31 207.01 0) (mirror x) (unit 1)
-    (in_bom yes) (on_board yes)
-    (property "Reference" "U1" (id 0) (at 67.31 212.09 0))
-    (property "Value" "LM833" (id 1) (at 67.31 214.63 0))
-    (property "Footprint" "Package_DIP:DIP-8_W7.62mm_Socket_LongPads" (id 2) (at 67.31 207.01 0)
-      (effects (font (size 1.27 1.27)) hide)
-    )
-    (property "Datasheet" "~" (id 3) (at 67.31 207.01 0)
-      (effects (font (size 1.27 1.27)) hide)
-    )
-    (pin "1")
-    (pin "2")
-    (pin "3")
   )
   (symbol (lib_id "Device:Opamp_Dual") (at 476.25 78.74 180) (unit 1)
@@
       (reference "TP29") (unit 1) (value "Vpreamp_R") (footprint "TestPoint:TestPoint_Keystone_5000-5004_Miniature")
     )
+    (path "/d783e9b2-f9eb-4b61-ab93-f012906accf8"
+      (reference "U1") (unit 1) (value "LM833") (footprint "Package_DIP:DIP-8_W7.62mm_Socket_LongPads")
+    )
     (path "/dcf9856d-8e58-482b-ac3e-ed7ca9899b4c"
-      (reference "U1") (unit 1) (value "LM833") (footprint "Package_DIP:DIP-8_W7.62mm_Socket_LongPads")
-    )
-    (path "/d783e9b2-f9eb-4b61-ab93-f012906accf8"
       (reference "U1") (unit 2) (value "LM833") (footprint "Package_DIP:DIP-8_W7.62mm_Socket_LongPads")
     )
